Commit message: Update UFACTORY adapter for reforge-core 2.0.15

File: src/robot/example_usage/kinecal/uf850_custom_tool.urdf (robot description, URDF)
Before this commit: robot uf850, 8 links, 7 joints
Links:
- added link custom_tool, mass 0.35; collision cylinder length=0.15 radius=0.02; visual cylinder length=0.15 radius=0.02
Joints:
- added joint joint_custom_tool: type fixed, parent link_eef, child custom_tool, origin xyz=0 0 0 rpy=0 0 0
