Commit message: Changed URDF to use base/shoulder convention instead of shoulder_pan/shoulder_joint

File: src/robot/urdf/ur5e.urdf (robot description, URDF)
Before this commit: robot ur5e, 11 links, 10 joints
Joints:
- removed joint shoulder_lift_joint
- removed joint shoulder_pan_joint
- added joint base_joint: type revolute, parent base_link_inertia, child shoulder_link, origin xyz=0.0 0.0 0.1625 rpy=0.0 0.0 0.0, axis 0 0 1, limit lower=-6.283185307179586 upper=6.283185307179586 effort=150.0 velocity=3.141592653589793
- added joint shoulder_joint: type revolute, parent shoulder_link, child upper_arm_link, origin xyz=0.0 0.0 0.0 rpy=1.570796327 0.0 0.0, axis 0 0 1, limit lower=-6.283185307179586 upper=6.283185307179586 effort=150.0 velocity=3.141592653589793

Commit message: Revert change, as Part 2 requires that naming convention

File: src/robot/urdf/ur5e.urdf (robot description, URDF)
Before this commit: robot ur5e, 11 links, 10 joints
Joints:
- removed joint base_joint
- removed joint shoulder_joint
- added joint shoulder_lift_joint: type revolute, parent shoulder_link, child upper_arm_link, origin xyz=0.0 0.0 0.0 rpy=1.570796327 0.0 0.0, axis 0 0 1, limit lower=-6.283185307179586 upper=6.283185307179586 effort=150.0 velocity=3.141592653589793
- added joint shoulder_pan_joint: type revolute, parent base_link_inertia, child shoulder_link, origin xyz=0.0 0.0 0.1625 rpy=0.0 0.0 0.0, axis 0 0 1, limit lower=-6.283185307179586 upper=6.283185307179586 effort=150.0 velocity=3.141592653589793
