Commit message: Changes for end-to-end pipeline testing

File: src/robot/urdf/axol-left.urdf (robot description, URDF)
Before this commit: robot assembly, 20 links, 19 joints
Links:
- link base: geometry collision mesh filename=/home/reforge/Desktop/almond-integration/reforge-interface/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 scale=1 1 1; visual mesh filename=/home/reforge/Desktop/almond-integration/reforge-interface/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 scale=1 1 1
- link left_e1: geometry collision mesh filename=/home/reforge/Desktop/almond-integration/reforge-interface/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 scale=1 1 1; visual mesh filename=/home/reforge/Desktop/almond-integration/reforge-interface/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 scale=1 1 1
- link left_e2: geometry collision mesh filename=/home/reforge/Desktop/almond-integration/reforge-interface/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 scale=1 1 1; visual mesh filename=/home/reforge/Desktop/almond-integration/reforge-interface/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 scale=1 1 1
- link left_gripper: geometry collision mesh filename=/home/reforge/Desktop/almond-integration/reforge-interface/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 scale=1 1 1; visual mesh filename=/home/reforge/Desktop/almond-integration/reforge-interface/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 scale=1 1 1
- link left_s2: geometry collision mesh filename=/home/reforge/Desktop/almond-integration/reforge-interface/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 scale=1 1 1; visual mesh filename=/home/reforge/Desktop/almond-integration/reforge-interface/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 scale=1 1 1
- link left_s3: geometry collision mesh filename=/home/reforge/Desktop/almond-integration/reforge-interface/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 scale=1 1 1; visual mesh filename=/home/reforge/Desktop/almond-integration/reforge-interface/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 scale=1 1 1
- link left_w0: geometry collision mesh filename=/home/reforge/Desktop/almond-integration/reforge-interface/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 scale=1 1 1; visual mesh filename=/home/reforge/Desktop/almond-integration/reforge-interface/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 scale=1 1 1
- link left_w1: geometry collision mesh filename=/home/reforge/Desktop/almond-integration/reforge-interface/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 scale=1 1 1; visual mesh filename=/home/reforge/Desktop/almond-integration/reforge-interface/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 scale=1 1 1
- link left_w2: geometry collision mesh filename=/home/reforge/Desktop/almond-integration/reforge-interface/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 scale=1 1 1; visual mesh filename=/home/reforge/Desktop/almond-integration/reforge-interface/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 scale=1 1 1
- link right_e1: geometry collision mesh filename=/home/reforge/Desktop/almond-integration/reforge-interface/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 scale=1 1 1; visual mesh filename=/home/reforge/Desktop/almond-integration/reforge-interface/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 scale=1 1 1
- link right_e2: geometry collision mesh filename=/home/reforge/Desktop/almond-integration/reforge-interface/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 scale=1 1 1; visual mesh filename=/home/reforge/Desktop/almond-integration/reforge-interface/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 scale=1 1 1
- link right_gripper: geometry collision mesh filename=/home/reforge/Desktop/almond-integration/reforge-interface/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 scale=1 1 1; visual mesh filename=/home/reforge/Desktop/almond-integration/reforge-interface/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 scale=1 1 1
- link right_s2: geometry collision mesh filename=/home/reforge/Desktop/almond-integration/reforge-interface/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 scale=1 1 1; visual mesh filename=/home/reforge/Desktop/almond-integration/reforge-interface/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 scale=1 1 1
- link right_s3: geometry collision mesh filename=/home/reforge/Desktop/almond-integration/reforge-interface/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 scale=1 1 1; visual mesh filename=/home/reforge/Desktop/almond-integration/reforge-interface/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 scale=1 1 1
- link right_w0: geometry collision mesh filename=/home/reforge/Desktop/almond-integration/reforge-interface/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 scale=1 1 1; visual mesh filename=/home/reforge/Desktop/almond-integration/reforge-interface/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 scale=1 1 1
- link right_w1: geometry collision mesh filename=/home/reforge/Desktop/almond-integration/reforge-interface/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 scale=1 1 1; visual mesh filename=/home/reforge/Desktop/almond-integration/reforge-interface/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 scale=1 1 1
- link right_w2: geometry collision mesh filename=/home/reforge/Desktop/almond-integration/reforge-interface/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 scale=1 1 1; visual mesh filename=/home/reforge/Desktop/almond-integration/reforge-interface/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 scale=1 1 1
- link s1: geometry collision mesh filename=/home/reforge/Desktop/almond-integration/reforge-interface/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 scale=1 1 1; visual mesh filename=/home/reforge/Desktop/almond-integration/reforge-interface/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 scale=1 1 1

File: src/robot/urdf/axol-right.urdf (robot description, URDF)
Before this commit: robot assembly, 20 links, 19 joints
Links:
- link base: geometry collision mesh filename=/home/reforge/Desktop/almond-integration/reforge-interface/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 scale=1 1 1; visual mesh filename=/home/reforge/Desktop/almond-integration/reforge-interface/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 scale=1 1 1
- link left_e1: geometry collision mesh filename=/home/reforge/Desktop/almond-integration/reforge-interface/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 scale=1 1 1; visual mesh filename=/home/reforge/Desktop/almond-integration/reforge-interface/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 scale=1 1 1
- link left_e2: geometry collision mesh filename=/home/reforge/Desktop/almond-integration/reforge-interface/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 scale=1 1 1; visual mesh filename=/home/reforge/Desktop/almond-integration/reforge-interface/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 scale=1 1 1
- link left_gripper: geometry collision mesh filename=/home/reforge/Desktop/almond-integration/reforge-interface/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 scale=1 1 1; visual mesh filename=/home/reforge/Desktop/almond-integration/reforge-interface/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 scale=1 1 1
- link left_s2: geometry collision mesh filename=/home/reforge/Desktop/almond-integration/reforge-interface/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 scale=1 1 1; visual mesh filename=/home/reforge/Desktop/almond-integration/reforge-interface/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 scale=1 1 1
- link left_s3: geometry collision mesh filename=/home/reforge/Desktop/almond-integration/reforge-interface/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 scale=1 1 1; visual mesh filename=/home/reforge/Desktop/almond-integration/reforge-interface/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 scale=1 1 1
- link left_w0: geometry collision mesh filename=/home/reforge/Desktop/almond-integration/reforge-interface/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 scale=1 1 1; visual mesh filename=/home/reforge/Desktop/almond-integration/reforge-interface/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 scale=1 1 1
- link left_w1: geometry collision mesh filename=/home/reforge/Desktop/almond-integration/reforge-interface/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 scale=1 1 1; visual mesh filename=/home/reforge/Desktop/almond-integration/reforge-interface/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 scale=1 1 1
- link left_w2: geometry collision mesh filename=/home/reforge/Desktop/almond-integration/reforge-interface/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 scale=1 1 1; visual mesh filename=/home/reforge/Desktop/almond-integration/reforge-interface/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 scale=1 1 1
- link right_e1: geometry collision mesh filename=/home/reforge/Desktop/almond-integration/reforge-interface/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 scale=1 1 1; visual mesh filename=/home/reforge/Desktop/almond-integration/reforge-interface/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 scale=1 1 1
- link right_e2: geometry collision mesh filename=/home/reforge/Desktop/almond-integration/reforge-interface/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 scale=1 1 1; visual mesh filename=/home/reforge/Desktop/almond-integration/reforge-interface/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 scale=1 1 1
- link right_gripper: geometry collision mesh filename=/home/reforge/Desktop/almond-integration/reforge-interface/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 scale=1 1 1; visual mesh filename=/home/reforge/Desktop/almond-integration/reforge-interface/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 scale=1 1 1
- link right_s2: geometry collision mesh filename=/home/reforge/Desktop/almond-integration/reforge-interface/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 scale=1 1 1; visual mesh filename=/home/reforge/Desktop/almond-integration/reforge-interface/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 scale=1 1 1
- link right_s3: geometry collision mesh filename=/home/reforge/Desktop/almond-integration/reforge-interface/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 scale=1 1 1; visual mesh filename=/home/reforge/Desktop/almond-integration/reforge-interface/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 scale=1 1 1
- link right_w0: geometry collision mesh filename=/home/reforge/Desktop/almond-integration/reforge-interface/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 scale=1 1 1; visual mesh filename=/home/reforge/Desktop/almond-integration/reforge-interface/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 scale=1 1 1
- link right_w1: geometry collision mesh filename=/home/reforge/Desktop/almond-integration/reforge-interface/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 scale=1 1 1; visual mesh filename=/home/reforge/Desktop/almond-integration/reforge-interface/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 scale=1 1 1
- link right_w2: geometry collision mesh filename=/home/reforge/Desktop/almond-integration/reforge-interface/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 scale=1 1 1; visual mesh filename=/home/reforge/Desktop/almond-integration/reforge-interface/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 scale=1 1 1
- link s1: geometry collision mesh filename=/home/reforge/Desktop/almond-integration/reforge-interface/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 scale=1 1 1; visual mesh filename=/home/reforge/Desktop/almond-integration/reforge-interface/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 scale=1 1 1

Commit message: Use explicit calibration options and relative paths in URDF meshes

File: src/robot/urdf/axol-left.urdf (robot description, URDF)
Before this commit: robot assembly, 20 links, 19 joints
Links:
- link base: geometry collision mesh filename=meshes/Base.stl scale=1 1 1; visual mesh filename=meshes/Base.stl scale=1 1 1
- link left_e1: geometry collision mesh filename=meshes/Left_E1.stl scale=1 1 1; visual mesh filename=meshes/Left_E1.stl scale=1 1 1
- link left_e2: geometry collision mesh filename=meshes/Left_E2.stl scale=1 1 1; visual mesh filename=meshes/Left_E2.stl scale=1 1 1
- link left_gripper: geometry collision mesh filename=meshes/Left_Gripper.stl scale=1 1 1; visual mesh filename=meshes/Left_Gripper.stl scale=1 1 1
- link left_s2: geometry collision mesh filename=meshes/Left_S2.stl scale=1 1 1; visual mesh filename=meshes/Left_S2.stl scale=1 1 1
- link left_s3: geometry collision mesh filename=meshes/Left_S3.stl scale=1 1 1; visual mesh filename=meshes/Left_S3.stl scale=1 1 1
- link left_w0: geometry collision mesh filename=meshes/Left_W0.stl scale=1 1 1; visual mesh filename=meshes/Left_W0.stl scale=1 1 1
- link left_w1: geometry collision mesh filename=meshes/Left_W1.stl scale=1 1 1; visual mesh filename=meshes/Left_W1.stl scale=1 1 1
- link left_w2: geometry collision mesh filename=meshes/Left_W2.stl scale=1 1 1; visual mesh filename=meshes/Left_W2.stl scale=1 1 1
- link right_e1: geometry collision mesh filename=meshes/Right_E1.stl scale=1 1 1; visual mesh filename=meshes/Right_E1.stl scale=1 1 1
- link right_e2: geometry collision mesh filename=meshes/Right_E2.stl scale=1 1 1; visual mesh filename=meshes/Right_E2.stl scale=1 1 1
- link right_gripper: geometry collision mesh filename=meshes/Right_Gripper.stl scale=1 1 1; visual mesh filename=meshes/Right_Gripper.stl scale=1 1 1
- link right_s2: geometry collision mesh filename=meshes/Right_S2.stl scale=1 1 1; visual mesh filename=meshes/Right_S2.stl scale=1 1 1
- link right_s3: geometry collision mesh filename=meshes/Right_S3.stl scale=1 1 1; visual mesh filename=meshes/Right_S3.stl scale=1 1 1
- link right_w0: geometry collision mesh filename=meshes/Right_W0.stl scale=1 1 1; visual mesh filename=meshes/Right_W0.stl scale=1 1 1
- link right_w1: geometry collision mesh filename=meshes/Right_W1.stl scale=1 1 1; visual mesh filename=meshes/Right_W1.stl scale=1 1 1
- link right_w2: geometry collision mesh filename=meshes/Right_W2.stl scale=1 1 1; visual mesh filename=meshes/Right_W2.stl scale=1 1 1
- link s1: geometry collision mesh filename=meshes/S1.stl scale=1 1 1; visual mesh filename=meshes/S1.stl scale=1 1 1

File: src/robot/urdf/axol-right.urdf (robot description, URDF)
Before this commit: robot assembly, 20 links, 19 joints
Links:
- link base: geometry collision mesh filename=meshes/Base.stl scale=1 1 1; visual mesh filename=meshes/Base.stl scale=1 1 1
- link left_e1: geometry collision mesh filename=meshes/Left_E1.stl scale=1 1 1; visual mesh filename=meshes/Left_E1.stl scale=1 1 1
- link left_e2: geometry collision mesh filename=meshes/Left_E2.stl scale=1 1 1; visual mesh filename=meshes/Left_E2.stl scale=1 1 1
- link left_gripper: geometry collision mesh filename=meshes/Left_Gripper.stl scale=1 1 1; visual mesh filename=meshes/Left_Gripper.stl scale=1 1 1
- link left_s2: geometry collision mesh filename=meshes/Left_S2.stl scale=1 1 1; visual mesh filename=meshes/Left_S2.stl scale=1 1 1
- link left_s3: geometry collision mesh filename=meshes/Left_S3.stl scale=1 1 1; visual mesh filename=meshes/Left_S3.stl scale=1 1 1
- link left_w0: geometry collision mesh filename=meshes/Left_W0.stl scale=1 1 1; visual mesh filename=meshes/Left_W0.stl scale=1 1 1
- link left_w1: geometry collision mesh filename=meshes/Left_W1.stl scale=1 1 1; visual mesh filename=meshes/Left_W1.stl scale=1 1 1
- link left_w2: geometry collision mesh filename=meshes/Left_W2.stl scale=1 1 1; visual mesh filename=meshes/Left_W2.stl scale=1 1 1
- link right_e1: geometry collision mesh filename=meshes/Right_E1.stl scale=1 1 1; visual mesh filename=meshes/Right_E1.stl scale=1 1 1
- link right_e2: geometry collision mesh filename=meshes/Right_E2.stl scale=1 1 1; visual mesh filename=meshes/Right_E2.stl scale=1 1 1
- link right_gripper: geometry collision mesh filename=meshes/Right_Gripper.stl scale=1 1 1; visual mesh filename=meshes/Right_Gripper.stl scale=1 1 1
- link right_s2: geometry collision mesh filename=meshes/Right_S2.stl scale=1 1 1; visual mesh filename=meshes/Right_S2.stl scale=1 1 1
- link right_s3: geometry collision mesh filename=meshes/Right_S3.stl scale=1 1 1; visual mesh filename=meshes/Right_S3.stl scale=1 1 1
- link right_w0: geometry collision mesh filename=meshes/Right_W0.stl scale=1 1 1; visual mesh filename=meshes/Right_W0.stl scale=1 1 1
- link right_w1: geometry collision mesh filename=meshes/Right_W1.stl scale=1 1 1; visual mesh filename=meshes/Right_W1.stl scale=1 1 1
- link right_w2: geometry collision mesh filename=meshes/Right_W2.stl scale=1 1 1; visual mesh filename=meshes/Right_W2.stl scale=1 1 1
- link s1: geometry collision mesh filename=meshes/S1.stl scale=1 1 1; visual mesh filename=meshes/S1.stl scale=1 1 1
