Commit message: Update wxai_follower.urdf

File: src/robot/urdf/trossen/wxai_follower.urdf (robot description, URDF)
Before this commit: robot wxai, 23 links, 22 joints
Links:
- removed link tool0
- added link ee_gripper_link
- link base_link: geometry collision mesh filename=meshes/base_link.stl; visual mesh filename=meshes/base_link.stl
- link camera_link: geometry collision box size=0.023 0.042 0.042; visual mesh filename=meshes/d405.stl scale=0.001 0.001 0.001
- link camera_mount_d405: geometry collision mesh filename=meshes/camera_mount_d405.stl; visual mesh filename=meshes/camera_mount_d405.stl
- link carriage_left: geometry collision mesh filename=meshes/carriage_left.stl; visual mesh filename=meshes/carriage_left.stl
- link carriage_right: geometry collision mesh filename=meshes/carriage_right.stl; visual mesh filename=meshes/carriage_right.stl
- link gripper_left: geometry collision mesh filename=meshes/gripper_left.stl; visual mesh filename=meshes/gripper_left.stl
- link gripper_right: geometry collision mesh filename=meshes/gripper_right.stl; visual mesh filename=meshes/gripper_right.stl
- link link_1: geometry collision mesh filename=meshes/link_1.stl; visual mesh filename=meshes/link_1.stl
- link link_2: geometry collision mesh filename=meshes/link_2.stl; visual mesh filename=meshes/link_2.stl
- link link_3: geometry collision mesh filename=meshes/link_3.stl; visual mesh filename=meshes/link_3.stl
- link link_4: geometry collision mesh filename=meshes/link_4.stl; visual mesh filename=meshes/link_4.stl
- link link_5: geometry collision mesh filename=meshes/link_5.stl; visual mesh filename=meshes/link_5.stl
- link link_6: mass 0.83441558 -> 0.55469347; geometry collision mesh filename=meshes/link_6.stl; visual mesh filename=meshes/link_6.stl
Joints:
- joint camera_mount_joint: axis (none) -> 0 0 0
- joint ee_gripper: axis (none) -> 1 0 0; child tool0 -> ee_gripper_link
- joint left_carriage_joint: axis (none) -> 0 1 0; limit (none) -> lower=0.0 upper=0.044 effort=400.0 velocity=0.0875; type fixed -> prismatic
- joint left_gripper_joint: axis (none) -> 0 0 0
- joint right_carriage_joint: axis (none) -> 0 -1 0; limit (none) -> lower=0.0 upper=0.044 effort=400.0 velocity=0.0875; mimic (none) -> joint=left_carriage_joint; type fixed -> prismatic
- joint right_gripper_joint: axis (none) -> 0 0 0

Commit message: Refactor wxai_follower URDF for mesh paths and joints
Updated mesh file paths to include 'wxai' directory and modified joint types for carriages from 'prismatic' to 'fixed'. Added centered_fixture link for calibration.

File: src/robot/urdf/trossen/wxai_follower.urdf (robot description, URDF)
Before this commit: robot wxai, 23 links, 22 joints
Links:
- removed link ee_gripper_link
- added link centered_fixture
- link base_link: geometry collision mesh filename=meshes/wxai/base_link.stl; visual mesh filename=meshes/wxai/base_link.stl
- link camera_link: geometry collision box size=0.023 0.042 0.042; visual mesh filename=meshes/peripherals/d405.stl scale=0.001 0.001 0.001
- link camera_mount_d405: geometry collision mesh filename=meshes/wxai/camera_mount_d405.stl; visual mesh filename=meshes/wxai/camera_mount_d405.stl
- link carriage_left: geometry collision mesh filename=meshes/wxai/carriage_left.stl; visual mesh filename=meshes/wxai/carriage_left.stl
- link carriage_right: geometry collision mesh filename=meshes/wxai/carriage_right.stl; visual mesh filename=meshes/wxai/carriage_right.stl
- link gripper_left: geometry collision mesh filename=meshes/wxai/gripper_left.stl; visual mesh filename=meshes/wxai/gripper_left.stl
- link gripper_right: geometry collision mesh filename=meshes/wxai/gripper_right.stl; visual mesh filename=meshes/wxai/gripper_right.stl
- link link_1: geometry collision mesh filename=meshes/wxai/link_1.stl; visual mesh filename=meshes/wxai/link_1.stl
- link link_2: geometry collision mesh filename=meshes/wxai/link_2.stl; visual mesh filename=meshes/wxai/link_2.stl
- link link_3: geometry collision mesh filename=meshes/wxai/link_3.stl; visual mesh filename=meshes/wxai/link_3.stl
- link link_4: geometry collision mesh filename=meshes/wxai/link_4.stl; visual mesh filename=meshes/wxai/link_4.stl
- link link_5: geometry collision mesh filename=meshes/wxai/link_5.stl; visual mesh filename=meshes/wxai/link_5.stl
- link link_6: mass 0.55469347 -> 0.83441558; geometry collision mesh filename=meshes/wxai/link_6.stl; visual mesh filename=meshes/wxai/link_6.stl
Joints:
- removed joint ee_gripper
- added joint centered_fixture_joint: type fixed, parent link_6, child centered_fixture, origin xyz=0.0865 0 0 rpy=0 0 0
- joint camera_mount_joint: axis 0 0 0 -> (none)
- joint left_carriage_joint: axis 0 1 0 -> (none); limit lower=0.0 upper=0.044 effort=400.0 velocity=0.0875 -> (none); type prismatic -> fixed
- joint left_gripper_joint: axis 0 0 0 -> (none)
- joint right_carriage_joint: axis 0 -1 0 -> (none); limit lower=0.0 upper=0.044 effort=400.0 velocity=0.0875 -> (none); mimic joint=left_carriage_joint -> (none); type prismatic -> fixed
- joint right_gripper_joint: axis 0 0 0 -> (none)

Commit message: Add fixed joint and tool link to URDF
Adding additional link for the Kinecal

File: src/robot/urdf/trossen/wxai_follower.urdf (robot description, URDF)
Before this commit: robot wxai, 23 links, 22 joints
Links:
- added link tool0
Joints:
- added joint ee_gripper: type fixed, parent link_6, child tool0, origin xyz=0.156062 0 0 rpy=0 0 0
