Commit message: Move Standard Bots RO1 URDF into urdf/RO1 and add its meshes
The Standard Bots RO1 URDF and its visual/collision meshes now live together
under src/robot/urdf/RO1, matching the layout already validated in
reforge-core (src/robot/urdf/standardbots + src/robot/urdf/meshes there,
collapsed into one directory here since the meshes have nowhere else to live
in this repo yet).

- src/robot/urdf/modelone.urdf -> src/robot/urdf/RO1/modelone.urdf.
- Added src/robot/urdf/RO1/meshes/: 14 STL files (7 links x visual/collision),
  copied byte-for-byte from reforge-core's flattened, already-renamed set and
  verified with cmp against every file.
- Rewrote modelone.urdf's 14 mesh <mesh filename> references from
  package://standard_bots_description/meshes/sbot/{visual,collision}/<link>.STL
  to the relative meshes/<link>_<kind>.STL, for the same reason reforge-core
  made this change: CollisionModel passes the URDF's own directory as
  Pinocchio's package_dirs and does not consult ROS_PACKAGE_PATH, so a
  package:// URI never resolved here. Documented in a new
  urdf/RO1/meshes/README.md, adapted from reforge-core's.
- robot_interface.py: URDF_PATH now points at urdf/RO1/modelone.urdf. This is
  the only reference to the old path in the repo.
- pyproject.toml / MANIFEST.in: added an uppercase *.STL pattern alongside the
  existing lowercase *.stl. The repo had no STL files before this change, so
  the case-sensitive glob was untested; without this fix a non-editable
  install would silently drop the new meshes from the built package.

Verified: buildModelFromUrdf + buildGeomFromUrdf(..., package_dirs=[urdf_dir])
resolves and loads all 7 visual and 7 collision meshes from the new location
(the same mechanism CollisionModel uses). robot_interface.py's own
files("robot").joinpath(URDF_PATH) resolution finds the moved file. Full test
suite (11 tests) passes.

Not carried over: the upstream package.xml, which the meshes' own README
notes declares the package Proprietary even though a mirror's root license is
MIT.

Co-Authored-By: Claude Opus 5 <noreply@anthropic.com>

File: src/robot/urdf/RO1/modelone.urdf (robot description, URDF)
Before this commit: robot sbot, 9 links, 8 joints
Links:
- link base_link: geometry collision mesh filename=meshes/base_link_collision.STL; visual mesh filename=meshes/base_link_visual.STL
- link forearm_link: geometry collision mesh filename=meshes/forearm_link_collision.STL; visual mesh filename=meshes/forearm_link_visual.STL
- link shoulder_link: geometry collision mesh filename=meshes/shoulder_link_collision.STL; visual mesh filename=meshes/shoulder_link_visual.STL
- link upper_arm_link: geometry collision mesh filename=meshes/upper_arm_link_collision.STL; visual mesh filename=meshes/upper_arm_link_visual.STL
- link wrist_1_link: geometry collision mesh filename=meshes/wrist_1_link_collision.STL; visual mesh filename=meshes/wrist_1_link_visual.STL
- link wrist_2_link: geometry collision mesh filename=meshes/wrist_2_link_collision.STL; visual mesh filename=meshes/wrist_2_link_visual.STL
- link wrist_3_link: geometry collision mesh filename=meshes/wrist_3_link_collision.STL; visual mesh filename=meshes/wrist_3_link_visual.STL
