Commit message: Fix Yaskawa model frames and KineCal config

File: src/robot/urdf/NEX07C00/NEX07C00.urdf (robot description, URDF)
Before this commit: robot NEX07C00, 9 links, 8 joints
Links:
- removed link B
- removed link L
- removed link R
- removed link S
- removed link T
- removed link U
- added link B_link; collision mesh filename=collision/Collision_5_1.obj scale=0.001000 0.001000 0.001000; collision mesh filename=collision/Collision_5_2.obj scale=0.001000 0.001000 0.001000
- added link L_link; collision mesh filename=collision/Collision_2_1.obj scale=0.001000 0.001000 0.001000; collision mesh filename=collision/Collision_2_2.obj scale=0.001000 0.001000 0.001000
- added link R_link; collision mesh filename=collision/Collision_4_1.obj scale=0.001000 0.001000 0.001000; collision mesh filename=collision/Collision_4_2.obj scale=0.001000 0.001000 0.001000
- added link S_link; collision mesh filename=collision/Collision_1_1.obj scale=0.001000 0.001000 0.001000; collision mesh filename=collision/Collision_1_2.obj scale=0.001000 0.001000 0.001000
- added link T_link; collision mesh filename=collision/Collision_6_1.obj scale=0.001000 0.001000 0.001000; collision mesh filename=collision/Collision_6_2.obj scale=0.001000 0.001000 0.001000
- added link U_link; collision mesh filename=collision/Collision_3_1.obj scale=0.001000 0.001000 0.001000; collision mesh filename=collision/Collision_3_2.obj scale=0.001000 0.001000 0.001000
- added link tool0
Joints:
- added joint flange-tool0: type fixed, parent flange, child tool0, origin xyz=0 0 0 rpy=0 0 0
- joint B: child B -> B_link; parent R -> R_link
- joint L: child L -> L_link; parent S -> S_link
- joint R: child R -> R_link; parent U -> U_link
- joint S: child S -> S_link
- joint T: child T -> T_link; parent B -> B_link
- joint T-flange: parent T -> T_link
- joint U: child U -> U_link; parent L -> L_link

Commit message: Update NEX07C00 to account for 0.33m offset of the base joint

File: src/robot/urdf/NEX07C00/NEX07C00.urdf (robot description, URDF)
Before this commit: robot NEX07C00, 10 links, 9 joints
Joints:
- removed joint BASE-base
- added joint base-BASE: type fixed, parent base, child BASE, origin xyz=0.000000 0.000000 -0.330000 rpy=0.000000 0.000000 0.000000
